Commit message: angle of light param

File: sp_crazyflie_gazebo/models/rotors_description/urdf/crazyflie_base.xacro (robot description, xacro)
@@ -9,5 +9,6 @@
   <xacro:arg name='name' default='crazyflie' />
   <xacro:arg name='enable_wind' default='$(arg enable_wind)' />
-  <xacro:arg name='enable_light' default='true' />
+  <xacro:arg name='light_enable' default='true' />
+  <xacro:arg name='light_angle' default='${3.14/6}' />
   <!-- The following causes segfault with multiple vehicles if defaults to true!!! -->
   <xacro:arg name='enable_logging' default='false' />
@@ -25,5 +26,5 @@
   </xacro:if>
   <xacro:if value="$(arg enable_light)">
-    <xacro:spotlight_macro namespace="${namespace}" parent_link="base_link">
+    <xacro:spotlight_macro namespace="${namespace}" parent_link="base_link" angle="$(arg light_angle)">
     </xacro:spotlight_macro >
   </xacro:if>

File: sp_crazyflie_gazebo/models/rotors_description/urdf/vision_spot.xacro (robot description, xacro)
@@ -1,5 +1,5 @@
 <?xml version="1.0"?>
 <robot xmlns:xacro="http://ros.org/wiki/xacro">
-    <xacro:macro name="spotlight_macro" params="namespace parent_link
+    <xacro:macro name="spotlight_macro" params="namespace parent_link angle
      ">
         <joint name="${namespace}/spot_joint" type="fixed">
@@ -23,6 +23,6 @@
                 <cast_shadows>false</cast_shadows>
                 <spot>
-                    <inner_angle>1.04</inner_angle>
-                    <outer_angle>1.05</outer_angle>
+                    <inner_angle>${angle}</inner_angle>
+                    <outer_angle>${angle*1.01}</outer_angle>
                     <falloff>0.1</falloff>
                 </spot>
